Commit message: initial commit

File: urdf/ultra_udacity_bot.xacro (robot description, xacro)
@@ -1,6 +1,6 @@
 <?xml version='1.0'?>
 <robot name="ultra_udacity_bot" xmlns:xacro="http://www.ros.org/wiki/xacro">
-  <xacro:include filename="$(find udacity_bot)/urdf/ultra_udacity_bot.gazebo" />
-  <link name="robot_footprint"></link>
+  <xacro:include filename="$(find slam_project)/urdf/ultra_udacity_bot.gazebo" />
+  link name="robot_footprint"></link>
   <joint name="robot_footprint_joint" type="fixed">
     <origin xyz="0 0 0" rpy="0 0 0" />
@@ -23,5 +23,5 @@
       <origin xyz="0 0 -.08" rpy=" 0 0 210"/>
       <geometry>
-        <mesh filename="package://udacity_bot/meshes/udacity.dae"  scale=".45 .45 .45"/>
+        <mesh filename="package://slam_project/meshes/udacity.dae"  scale=".45 .45 .45"/>
       </geometry>
     </collision>
@@ -30,5 +30,5 @@
       <geometry>
       	<!-- model is 60 mm tall, 20 mm thick -->
-        <mesh filename="package://udacity_bot/meshes/udacity.dae" scale=".45 .45 .45"/>
+        <mesh filename="package://slam_project/meshes/udacity.dae" scale=".45 .45 .45"/>
       </geometry>
     </visual>
@@ -186,5 +186,5 @@
       <origin xyz="0 0 0" rpy=" 0 0 0"/>
       <geometry>
-        <mesh filename="package://udacity_bot/meshes/hokuyo.dae"/>
+        <mesh filename="package://slam_project/meshes/hokuyo.dae"/>
       </geometry>
     </visual>

Commit message: working configuration except for pointcloud projections into world frame

File: urdf/ultra_udacity_bot.xacro (robot description, xacro)
@@ -2,5 +2,5 @@
 <robot name="ultra_udacity_bot" xmlns:xacro="http://www.ros.org/wiki/xacro">
   <xacro:include filename="$(find slam_project)/urdf/ultra_udacity_bot.gazebo" />
-  link name="robot_footprint"></link>
+  <link name="robot_footprint"></link>
   <joint name="robot_footprint_joint" type="fixed">
     <origin xyz="0 0 0" rpy="0 0 0" />

Commit message: working code for mapping

File: urdf/ultra_udacity_bot.xacro (robot description, xacro)
@@ -161,4 +161,18 @@
     </visual>
   </link>
+  <!-- generate an optical frame
+      http://www.ros.org/reps/rep-0103.html#suffix-frames
+      so that ros and opencv can operate on the camera frame correctly
+      -->
+  <joint name="camera_optical_joint" type="fixed">
+    <!-- these values have to be these values otherwise the gazebo camera
+        image won't be aligned properly with the frame it is supposedly
+        originating from -->
+    <origin xyz="0 0 0" rpy="${-pi/2} 0 ${-pi/2}"/>
+    <parent link="camera"/>
+    <child link="camera_link_optical"/>
+  </joint>
+  <link name="camera_link_optical">
+  </link>
   <joint type="fixed" name="camera_joint">
     <origin xyz="0.15 0 -.03" rpy="0 0 0"/>
